File: pcb/plasma_modulator.sch (KiCad schematic (older format))
At the start: 85 parts, among them P1 CONN_01X03, P2 CONN_01X03, P3 CONN_01X06, P4 CONN_01X04, P5 RCA_1, Q1 MOSFET_N, Q2 MOSFET_N, Q3 MOSFET_N, Q4 MOSFET_N, SW1 SW_PUSH, SW2 SW_PUSH, SW3 SW_PUSH, U1 LD1117S33TR, U2 IXDD609SI, U3 IXDD609SI, U4 STM32F334K, U5 FAN7390, U6 LTC6101, U7 SN74LVC1T45, U8 SN74LVC1T45, U9 MIC5205, X1 13.56MHz

Commit message: plotted schematic and PCB layouts
Parts:
- C1, C10, C11, C12, C13, C14, C15, C16, C17, C18, C19, C2, C21, C22, C23, C24, C25, C26, C28, C29, C3, C30, C31, C32, C33, C34, C35, C36, C4, C5, C7, C8, C9: symbol C -> C-RESCUE-plasma_modulator
- D2, D3: symbol LED -> LED-RESCUE-plasma_modulator
- R1, R10, R11, R12, R13, R14, R15, R16, R17, R18, R19, R2, R20, R21, R3, R4, R5, R6, R7, R8, R9: symbol R -> R-RESCUE-plasma_modulator
